Commit message: Add sensors data

File: urdf/payload.urdf.xacro (robot description, xacro)
@@ -9,5 +9,13 @@
   <!-- <xacro:arg name="robot_xacro" default="$(find sparus2_description)/urdf/core.urdf.xacro"/> -->
   <xacro:arg name="robot_xacro" default="$(find xiroi_description)/urdf/core.urdf.xacro"/>
-  <!-- Load basic xiroi urdf -->
+  <!-- Load basic Xiroi urdf -->
   <xacro:include filename="$(arg robot_xacro)"/>
+  <!-- USBL
+  <xacro:add_to_base_link_no_mesh element="USBL">
+    <origin rpy="0 0 0" xyz="0.45 0 -0.13"/>
+  </xacro:add_to_base_link_no_mesh>-->
+  <!-- Cameras
+  <xacro:add_to_base_link_no_mesh element="multibeam">
+    <origin rpy="0 -${pi/2} ${pi}" xyz="0.5 0 0"/>
+  </xacro:add_to_base_link_no_mesh>-->
 </robot>

Commit message: andratx fieldtest usbl changes

File: urdf/payload.urdf.xacro (robot description, xacro)
@@ -11,8 +11,8 @@
   <!-- Load basic Xiroi urdf -->
   <xacro:include filename="$(arg robot_xacro)"/>
-  <!-- USBL
-  <xacro:add_to_base_link_no_mesh element="USBL">
-    <origin rpy="0 0 0" xyz="0.45 0 -0.13"/>
-  </xacro:add_to_base_link_no_mesh>-->
+  <!-- USBL -->
+  <!-- <xacro:add_to_base_link_no_mesh element="usbl">
+    <origin rpy="0 0 0" xyz="0.32 0 0.8"/>
+  </xacro:add_to_base_link_no_mesh> -->
   <!-- Cameras
   <xacro:add_to_base_link_no_mesh element="multibeam">
