Commit message: Added IMU frame

File: urdf/core.urdf.xacro (robot description, xacro)
@@ -22,12 +22,15 @@
   </xacro:add_to_base_link>
   <!-- IMU -->
-  <!-- TODO -->
   <xacro:add_to_base_link element="imu">
-    <origin rpy="0 0 0" xyz="0 0 0"/>
+    <origin rpy="${pi/2} 0 ${pi/2}" xyz="0.36377 -0.02093 -0.08490"/>
+  </xacro:add_to_base_link>
+  <!-- IMU aligned with robot axis.
+       This frame is where the data of the IMU filter is published -->
+  <xacro:add_to_base_link element="imu_filter">
+    <origin rpy="0 0 0" xyz="0.36377 -0.02093 -0.08490"/>
   </xacro:add_to_base_link>
   <!-- Pressure -->
-  <!-- TODO -->
   <xacro:add_to_base_link element="pressure">
-    <origin rpy="0 0 0" xyz="0 0 0"/>
+    <origin rpy="0 0 0" xyz="0.387 0 -0.33"/>
   </xacro:add_to_base_link>
   <!-- Thrusters -->

Commit message: Added dvl_altitude frame

File: urdf/core.urdf.xacro (robot description, xacro)
@@ -21,4 +21,7 @@
     <origin rpy="${pi} 0 ${3*pi/4}" xyz="-0.4145 0 0.1"/>
   </xacro:add_to_base_link>
+  <xacro:add_element element="dvl_altitude" parent="dvl">
+    <origin rpy="0 ${pi/2} 0" xyz="0 0 0"/>
+  </xacro:add_element>
   <!-- IMU -->
   <xacro:add_to_base_link element="imu">

Commit message: URDF corrected and change from 3ds to dae

File: urdf/core.urdf.xacro (robot description, xacro)
@@ -7,7 +7,7 @@
   <link name="$(arg robot_namespace)/base_link">
     <visual>
-      <origin rpy="-${pi/2} 0 0" xyz="0 0 0"/>
+      <origin rpy="0 0 0" xyz="0 0 0"/>
       <geometry>
-        <mesh filename="package://sparus2_description/meshes/sparus2.3ds" scale="1 1 1"/>
+        <mesh filename="package://sparus2_description/meshes/sparus2.dae" scale="1 1 1"/>
       </geometry>
     </visual>
@@ -15,9 +15,9 @@
   <!-- GPS -->
   <xacro:add_to_base_link_no_mesh element="gps">
-    <origin rpy="0 0 0" xyz="-0.39 0 -0.35"/>
+    <origin rpy="0 0 0" xyz="-0.39 0 -0.36"/>
   </xacro:add_to_base_link_no_mesh>
   <!-- DVL -->
   <xacro:add_to_base_link_no_mesh element="dvl">
-    <origin rpy="${pi} 0 ${3*pi/4}" xyz="-0.4145 0 0.1"/>
+    <origin rpy="${pi} 0 ${3*pi/4}" xyz="-0.4145 0 0.11"/>
   </xacro:add_to_base_link_no_mesh>
   <xacro:add_element_no_mesh element="dvl_altitude" parent="dvl">
@@ -31,19 +31,19 @@
        This frame is where the data of the IMU filter is published -->
   <xacro:add_to_base_link_no_mesh element="imu_filter">
-    <origin rpy="0 0 0" xyz="0.36377 -0.02093 -0.08490"/>
+    <origin rpy="0 0 0" xyz="0.36377 -0.02093 -0.0849"/>
   </xacro:add_to_base_link_no_mesh>
   <!-- Pressure -->
   <xacro:add_to_base_link_no_mesh element="pressure">
-    <origin rpy="0 0 0" xyz="0.387 0 -0.33"/>
+    <origin rpy="0 0 0" xyz="0.387 0 -0.033"/>
   </xacro:add_to_base_link_no_mesh>
   <!-- Thrusters -->
   <xacro:add_thruster_no_mesh thruster_id="0">
+    <origin xyz="0 0 0.08" rpy="0 0 0" />
+  </xacro:add_thruster_no_mesh>
+  <xacro:add_thruster_no_mesh thruster_id="1">
     <origin xyz="-0.59 0.17 0" rpy="0 0 ${pi}" />
   </xacro:add_thruster_no_mesh>
-  <xacro:add_thruster_no_mesh thruster_id="1">
+  <xacro:add_thruster_no_mesh thruster_id="2">
     <origin xyz="-0.59 -0.17 0" rpy="0 0 ${pi}" />
   </xacro:add_thruster_no_mesh>
-  <xacro:add_thruster_no_mesh thruster_id="2">
-    <origin xyz="0 0 0.08" rpy="0 0 0" />
-  </xacro:add_thruster_no_mesh>
 </robot>

Commit message: Change names

File: urdf/core.urdf.xacro (robot description, xacro)
@@ -9,5 +9,5 @@
       <origin rpy="0 0 0" xyz="0 0 0"/>
       <geometry>
-        <mesh filename="package://sparus2_description/meshes/sparus2.dae" scale="1 1 1"/>
+        <mesh filename="package://xiroi_description/meshes/xiroi.dae" scale="1 1 1"/>
       </geometry>
     </visual>

Commit message: Upload local changes: xiroi configuration

File: urdf/core.urdf.xacro (robot description, xacro)
@@ -13,29 +13,18 @@
     </visual>
   </link>
-  <!-- GPS -->
+  <!-- GPS
   <xacro:add_to_base_link_no_mesh element="gps">
     <origin rpy="0 0 0" xyz="-0.39 0 -0.36"/>
-  </xacro:add_to_base_link_no_mesh>
-  <!-- DVL -->
-  <xacro:add_to_base_link_no_mesh element="dvl">
-    <origin rpy="${pi} 0 ${3*pi/4}" xyz="-0.4145 0 0.11"/>
-  </xacro:add_to_base_link_no_mesh>
-  <xacro:add_element_no_mesh element="dvl_altitude" parent="dvl">
-    <origin rpy="0 ${pi/2} 0" xyz="0 0 0"/>
-  </xacro:add_element_no_mesh>
-  <!-- IMU -->
+  </xacro:add_to_base_link_no_mesh>-->
+  <!-- IMU
   <xacro:add_to_base_link_no_mesh element="imu">
     <origin rpy="${pi/2} 0 ${pi/2}" xyz="0.36377 -0.02093 -0.08490"/>
-  </xacro:add_to_base_link_no_mesh>
+  </xacro:add_to_base_link_no_mesh>-->
   <!-- IMU aligned with robot axis.
-       This frame is where the data of the IMU filter is published -->
+       This frame is where the data of the IMU filter is published
   <xacro:add_to_base_link_no_mesh element="imu_filter">
     <origin rpy="0 0 0" xyz="0.36377 -0.02093 -0.0849"/>
-  </xacro:add_to_base_link_no_mesh>
-  <!-- Pressure -->
-  <xacro:add_to_base_link_no_mesh element="pressure">
-    <origin rpy="0 0 0" xyz="0.387 0 -0.033"/>
-  </xacro:add_to_base_link_no_mesh>
-  <!-- Thrusters -->
+  </xacro:add_to_base_link_no_mesh>-->
+  <!-- Thrusters
   <xacro:add_thruster_no_mesh thruster_id="0">
     <origin xyz="0 0 0.08" rpy="0 0 0" />
@@ -46,4 +35,4 @@
   <xacro:add_thruster_no_mesh thruster_id="2">
     <origin xyz="-0.59 -0.17 0" rpy="0 0 ${pi}" />
-  </xacro:add_thruster_no_mesh>
+  </xacro:add_thruster_no_mesh>-->
 </robot>

File: urdf/payload.urdf.xacro (robot description, xacro)
@@ -1,4 +1,4 @@
 <?xml version="1.0"?>
-<robot name="sparus2" xmlns:xacro="http://www.ros.org/wiki/xacro">
+<robot name="xiroi" xmlns:xacro="http://www.ros.org/wiki/xacro">
   <!-- Arguments -->
   <!--
@@ -7,51 +7,7 @@
     xacro:arg name="robot_namespace" default="sparus2"/
   -->
-  <xacro:arg name="robot_xacro" default="$(find sparus2_description)/urdf/core.urdf.xacro"/>
-  <!-- Load basic Sparus 2 urdf -->
+  <!-- <xacro:arg name="robot_xacro" default="$(find sparus2_description)/urdf/core.urdf.xacro"/> -->
+  <xacro:arg name="robot_xacro" default="$(find xiroi_description)/urdf/core.urdf.xacro"/>
+  <!-- Load basic xiroi urdf -->
   <xacro:include filename="$(arg robot_xacro)"/>
-  <!-- Modem -->
-  <xacro:add_to_base_link_no_mesh element="modem">
-    <origin rpy="0 0 0" xyz="0.45 0 -0.13"/>
-  </xacro:add_to_base_link_no_mesh>
-  <!-- Multibeam -->
-  <xacro:add_to_base_link_no_mesh element="multibeam">
-    <origin rpy="0 -${pi/2} ${pi}" xyz="0.5 0 0"/>
-  </xacro:add_to_base_link_no_mesh>
-  <!-- Side Scan -->
-  <xacro:add_to_base_link_no_mesh element="sidescan_port">
-    <origin rpy="${pi/4} 0 0" xyz="0.22 -0.10129 0.05386"/>
-  </xacro:add_to_base_link_no_mesh>
-  <xacro:add_to_base_link_no_mesh element="sidescan_starbord">
-    <origin rpy="-${pi/4} 0 0" xyz="0.22 0.10129 0.05386"/>
-  </xacro:add_to_base_link_no_mesh>
-  <!-- Echosounders -->
-  <xacro:add_to_base_link_no_mesh element="echosounder11">
-    <origin rpy="0 0 ${pi/2}" xyz="0.6 0 0"/>
-  </xacro:add_to_base_link_no_mesh>
-  <xacro:add_to_base_link_no_mesh element="echosounder12">
-    <origin rpy="0 0 -${pi/4}" xyz="0.6 0 0"/>
-  </xacro:add_to_base_link_no_mesh>
-  <xacro:add_to_base_link_no_mesh element="echosounder13">
-    <origin rpy="0 0 ${pi/4}" xyz="0.6 0 0"/>
-  </xacro:add_to_base_link_no_mesh>
-  <xacro:add_to_base_link_no_mesh element="echosounder14">
-    <origin rpy="0 0 0" xyz="0.6 0 0"/>
-  </xacro:add_to_base_link_no_mesh>
-  <xacro:add_to_base_link_no_mesh element="echosounder15">
-    <origin rpy="0 -${pi/2} 0" xyz="0.6 0 0"/>
-  </xacro:add_to_base_link_no_mesh>
-  <!-- Guppy -->
-  <xacro:add_to_base_link_no_mesh element="guppy">
-    <origin rpy="0 0 0" xyz="0.7 0 0"/>
-  </xacro:add_to_base_link_no_mesh>
-  <!-- Micron -->
-  <xacro:add_to_base_link_no_mesh element="micron">
-    <!-- origin rpy="0 0 -${pi}" xyz="0.885 0 -0.21"/ --> <!-- horizontal -->
-    <origin rpy="0 0 -${pi}" xyz="0.7 0 -0.15"/> <!-- horizontal -->
-    <!-- origin rpy="${pi} ${pi/2} 0" xyz="0.918 0 -0.09"/ --> <!-- vertical -->
-  </xacro:add_to_base_link_no_mesh>
-  <!-- Profiler -->
-  <xacro:add_to_base_link_no_mesh element="profiler">
-    <origin rpy="0 ${pi} ${pi}" xyz="0.885 0 0.1"/>
-  </xacro:add_to_base_link_no_mesh>
 </robot>

Commit message: Add sensor tf parameters

File: urdf/core.urdf.xacro (robot description, xacro)
@@ -13,12 +13,12 @@
     </visual>
   </link>
-  <!-- GPS
+  <!-- GPS -->
   <xacro:add_to_base_link_no_mesh element="gps">
-    <origin rpy="0 0 0" xyz="-0.39 0 -0.36"/>
-  </xacro:add_to_base_link_no_mesh>-->
-  <!-- IMU
+    <origin rpy="0 0 0" xyz="-30 13 -25"/>
+  </xacro:add_to_base_link_no_mesh>
+  <!-- IMU -->
   <xacro:add_to_base_link_no_mesh element="imu">
-    <origin rpy="${pi/2} 0 ${pi/2}" xyz="0.36377 -0.02093 -0.08490"/>
-  </xacro:add_to_base_link_no_mesh>-->
+    <origin rpy="0 0 0" xyz="10 7 0"/>
+  </xacro:add_to_base_link_no_mesh>
   <!-- IMU aligned with robot axis.
        This frame is where the data of the IMU filter is published
@@ -26,13 +26,10 @@
     <origin rpy="0 0 0" xyz="0.36377 -0.02093 -0.0849"/>
   </xacro:add_to_base_link_no_mesh>-->
-  <!-- Thrusters
+  <!-- Thrusters -->
   <xacro:add_thruster_no_mesh thruster_id="0">
-    <origin xyz="0 0 0.08" rpy="0 0 0" />
+    <origin xyz="-50 50 30" rpy="0 0 0" />
   </xacro:add_thruster_no_mesh>
   <xacro:add_thruster_no_mesh thruster_id="1">
-    <origin xyz="-0.59 0.17 0" rpy="0 0 ${pi}" />
+    <origin xyz="-50 -50 30" rpy="0 0 0" />
   </xacro:add_thruster_no_mesh>
-  <xacro:add_thruster_no_mesh thruster_id="2">
-    <origin xyz="-0.59 -0.17 0" rpy="0 0 ${pi}" />
-  </xacro:add_thruster_no_mesh>-->
 </robot>

Commit message: tf changes

File: urdf/core.urdf.xacro (robot description, xacro)
@@ -15,9 +15,9 @@
   <!-- GPS -->
   <xacro:add_to_base_link_no_mesh element="gps">
-    <origin rpy="0 0 0" xyz="-30 13 -25"/>
+    <origin rpy="0 0 0" xyz="-0.30 0.13 -0.25"/>
   </xacro:add_to_base_link_no_mesh>
   <!-- IMU -->
   <xacro:add_to_base_link_no_mesh element="imu">
-    <origin rpy="0 0 0" xyz="10 7 0"/>
+    <origin rpy="0 0 0" xyz="0.10 0.7 0"/>
   </xacro:add_to_base_link_no_mesh>
   <!-- IMU aligned with robot axis.
@@ -27,9 +27,9 @@
   </xacro:add_to_base_link_no_mesh>-->
   <!-- Thrusters -->
-  <xacro:add_thruster_no_mesh thruster_id="0">
-    <origin xyz="-50 50 30" rpy="0 0 0" />
+  <xacro:add_thruster_no_mesh thruster_id="1">
+    <origin xyz="-0.50 0.50 0.30" rpy="0 0 0" />
   </xacro:add_thruster_no_mesh>
-  <xacro:add_thruster_no_mesh thruster_id="1">
-    <origin xyz="-50 -50 30" rpy="0 0 0" />
+  <xacro:add_thruster_no_mesh thruster_id="2">
+    <origin xyz="-0.50 -0.50 0.30" rpy="0 0 0" />
   </xacro:add_thruster_no_mesh>
 </robot>

Commit message: Remove devices

File: urdf/core.urdf.xacro (robot description, xacro)
@@ -15,9 +15,9 @@
   <!-- GPS -->
   <xacro:add_to_base_link_no_mesh element="gps">
-    <origin rpy="0 0 0" xyz="-0.30 0.13 -0.25"/>
+    <origin rpy="0 0 0" xyz="0.60 0.0 -1.0"/><!-- <origin rpy="0 0 0" xyz="-0.30 0.13 -0.25"/> -->
   </xacro:add_to_base_link_no_mesh>
   <!-- IMU -->
   <xacro:add_to_base_link_no_mesh element="imu">
-    <origin rpy="0 0 0" xyz="0.10 0.7 0"/>
+    <origin rpy="0 0 0" xyz="-0.20 -0.25 -0.67"/>
   </xacro:add_to_base_link_no_mesh>
   <!-- IMU aligned with robot axis.

Commit message: IMU TF

File: urdf/core.urdf.xacro (robot description, xacro)
@@ -19,5 +19,5 @@
   <!-- IMU -->
   <xacro:add_to_base_link_no_mesh element="imu">
-    <origin rpy="0 0 0" xyz="0.10 0.7 0"/>
+    <origin rpy="3.1416 0 1.5708" xyz="0.10 0.7 0"/>
   </xacro:add_to_base_link_no_mesh>
   <!-- IMU aligned with robot axis.

Commit message: update IMU TF

File: urdf/core.urdf.xacro (robot description, xacro)
@@ -19,5 +19,6 @@
   <!-- IMU -->
   <xacro:add_to_base_link_no_mesh element="imu">
-    <origin rpy="3.1416 0 1.5708" xyz="0.10 0.7 0"/>
+    <origin rpy="0 3.1416 1.5707" xyz="1 0 0"/>
+    <!-- <origin rpy="0 0 0" xyz="1 0 0"/> -->
   </xacro:add_to_base_link_no_mesh>
   <!-- IMU aligned with robot axis.

Commit message: Clean comments

File: urdf/core.urdf.xacro (robot description, xacro)
@@ -20,11 +20,5 @@
   <xacro:add_to_base_link_no_mesh element="imu">
     <origin rpy="0 3.1416 1.5707" xyz="1 0 0"/>
-    <!-- <origin rpy="0 0 0" xyz="1 0 0"/> -->
   </xacro:add_to_base_link_no_mesh>
-  <!-- IMU aligned with robot axis.
-       This frame is where the data of the IMU filter is published
-  <xacro:add_to_base_link_no_mesh element="imu_filter">
-    <origin rpy="0 0 0" xyz="0.36377 -0.02093 -0.0849"/>
-  </xacro:add_to_base_link_no_mesh>-->
   <!-- Thrusters -->
   <xacro:add_thruster_no_mesh thruster_id="1">

Commit message: fix urdf IMU tranform error

File: urdf/core.urdf.xacro (robot description, xacro)
@@ -19,5 +19,5 @@
   <!-- IMU -->
   <xacro:add_to_base_link_no_mesh element="imu">
-    <origin rpy="0 3.1416 1.5707" xyz="1 0 0"/>
+    <origin rpy="0 3.1416 3.1416" xyz="1 0 0"/>
   </xacro:add_to_base_link_no_mesh>
   <!-- Thrusters -->

Commit message: memsense IMU TF update

File: urdf/core.urdf.xacro (robot description, xacro)
@@ -19,5 +19,5 @@
   <!-- IMU -->
   <xacro:add_to_base_link_no_mesh element="imu">
-    <origin rpy="0 3.1416 3.1416" xyz="1 0 0"/>
+    <origin rpy="0 0 1.57" xyz="1 0 0"/>
   </xacro:add_to_base_link_no_mesh>
   <!-- Thrusters -->

Commit message: Xiroi pond trials changes

File: urdf/core.urdf.xacro (robot description, xacro)
@@ -19,5 +19,5 @@
   <!-- IMU -->
   <xacro:add_to_base_link_no_mesh element="imu">
-    <origin rpy="0 0 1.57" xyz="1 0 0"/>
+    <origin rpy="0 0 1.57" xyz="-0.1 -0.1 0"/>
   </xacro:add_to_base_link_no_mesh>
   <!-- Thrusters -->

Commit message: update IMU and GPS TF's

File: urdf/core.urdf.xacro (robot description, xacro)
@@ -15,9 +15,9 @@
   <!-- GPS -->
   <xacro:add_to_base_link_no_mesh element="gps">
-    <origin rpy="0 0 0" xyz="0.60 0.0 -1.0"/><!-- <origin rpy="0 0 0" xyz="-0.30 0.13 -0.25"/> -->
+    <origin rpy="0 0 0" xyz="0.60 0.5 -0.1"/><!-- <origin rpy="0 0 0" xyz="-0.30 0.13 -0.25"/> -->
   </xacro:add_to_base_link_no_mesh>
   <!-- IMU -->
   <xacro:add_to_base_link_no_mesh element="imu">
-    <origin rpy="0 0 1.57" xyz="-0.1 -0.1 0"/>
+    <origin rpy="0 0 -1.57" xyz="-0.35 0.1 -0.2"/>
   </xacro:add_to_base_link_no_mesh>
   <!-- Thrusters -->

Commit message: add usbl tf

File: urdf/core.urdf.xacro (robot description, xacro)
@@ -15,9 +15,13 @@
   <!-- GPS -->
   <xacro:add_to_base_link_no_mesh element="gps">
-    <origin rpy="0 0 0" xyz="0.60 0.5 -0.1"/><!-- <origin rpy="0 0 0" xyz="-0.30 0.13 -0.25"/> -->
+    <origin rpy="0 0 0" xyz="0.60 0.5 -0.1"/>
   </xacro:add_to_base_link_no_mesh>
   <!-- IMU -->
   <xacro:add_to_base_link_no_mesh element="imu">
     <origin rpy="0 0 -1.57" xyz="-0.35 0.1 -0.2"/>
+  </xacro:add_to_base_link_no_mesh>
+  <!-- USBL -->
+  <xacro:add_to_base_link_no_mesh element="usbl">
+    <origin rpy="0 0 0" xyz="0.60 0 0.9"/>
   </xacro:add_to_base_link_no_mesh>
   <!-- Thrusters -->

Commit message: Add USBL tf

File: urdf/core.urdf.xacro (robot description, xacro)
@@ -15,9 +15,13 @@
   <!-- GPS -->
   <xacro:add_to_base_link_no_mesh element="gps">
-    <origin rpy="0 0 0" xyz="0.60 0.5 -0.1"/><!-- <origin rpy="0 0 0" xyz="-0.30 0.13 -0.25"/> -->
+    <origin rpy="0 0 0" xyz="0.70 0.35 -0.1"/>
   </xacro:add_to_base_link_no_mesh>
   <!-- IMU -->
   <xacro:add_to_base_link_no_mesh element="imu">
     <origin rpy="0 0 -1.57" xyz="-0.35 0.1 -0.2"/>
+  </xacro:add_to_base_link_no_mesh>
+  <!-- USBL -->
+  <xacro:add_to_base_link_no_mesh element="usbl">
+    <origin rpy="0 0 0" xyz="0.32 0 0.8"/>
   </xacro:add_to_base_link_no_mesh>
   <!-- Thrusters -->

Commit message: tf usbl moved to payload.urdf

File: urdf/core.urdf.xacro (robot description, xacro)
@@ -20,9 +20,13 @@
   <xacro:add_to_base_link_no_mesh element="imu">
     <origin rpy="0 0 -1.57" xyz="-0.35 0.1 -0.2"/>
+    <!-- good_: -->
+    <!-- <origin rpy="0 0 3.14" xyz="-0.35 0.1 -0.2"/> -->
+    <!-- <origin rpy="2.5 3.14 0.25" xyz="-0.35 0.1 -0.2"/> -->
+    <!-- <origin rpy="3.14 0 0" xyz="-0.35 0.1 -0.2"/> -->
   </xacro:add_to_base_link_no_mesh>
   <!-- USBL -->
-  <xacro:add_to_base_link_no_mesh element="usbl">
+  <!-- <xacro:add_to_base_link_no_mesh element="usbl">
     <origin rpy="0 0 0" xyz="0.32 0 0.8"/>
-  </xacro:add_to_base_link_no_mesh>
+  </xacro:add_to_base_link_no_mesh> -->
   <!-- Thrusters -->
   <xacro:add_thruster_no_mesh thruster_id="1">

File: urdf/payload.urdf.xacro (robot description, xacro)
@@ -12,7 +12,7 @@
   <xacro:include filename="$(arg robot_xacro)"/>
   <!-- USBL -->
-  <!-- <xacro:add_to_base_link_no_mesh element="usbl">
+  <xacro:add_to_base_link_no_mesh element="usbl">
     <origin rpy="0 0 0" xyz="0.32 0 0.8"/>
-  </xacro:add_to_base_link_no_mesh> -->
+  </xacro:add_to_base_link_no_mesh>
   <!-- Cameras
   <xacro:add_to_base_link_no_mesh element="multibeam">

Commit message: update IMU according to the real position

File: urdf/core.urdf.xacro (robot description, xacro)
@@ -19,9 +19,10 @@
   <!-- IMU -->
   <xacro:add_to_base_link_no_mesh element="imu">
-    <origin rpy="0 0 -1.57" xyz="-0.35 0.1 -0.2"/>
-    <!-- good_: -->
-    <!-- <origin rpy="0 0 3.14" xyz="-0.35 0.1 -0.2"/> -->
-    <!-- <origin rpy="2.5 3.14 0.25" xyz="-0.35 0.1 -0.2"/> -->
-    <!-- <origin rpy="3.14 0 0" xyz="-0.35 0.1 -0.2"/> -->
+    <origin rpy="0 0 3.14" xyz="-0.35 0.1 -0.2"/>
+  </xacro:add_to_base_link_no_mesh>
+    <!-- IMU aligned with robot axis.
+       This frame is where the data of the IMU filter is published -->
+  <xacro:add_to_base_link_no_mesh element="imu_filter">
+    <origin rpy="0 0 0" xyz="-0.35 0.1 -0.2"/>
   </xacro:add_to_base_link_no_mesh>
   <!-- USBL -->

Commit message: upload xiroi.dae in order to visualize the robot morphology in simulations

File: urdf/core.urdf.xacro (robot description, xacro)
@@ -7,7 +7,7 @@
   <link name="$(arg robot_namespace)/base_link">
     <visual>
-      <origin rpy="0 0 0" xyz="0 0 0"/>
+      <origin rpy="-1.57 0 -1.57" xyz="-1 -1.2 0"/>
       <geometry>
-        <mesh filename="package://xiroi_description/meshes/xiroi.dae" scale="1 1 1"/>
+        <mesh filename="package://xiroi_description/meshes/xiroi.dae" scale="0.011 0.011 0.011"/>
       </geometry>
     </visual>

Commit message: imu_tfs

File: urdf/core.urdf.xacro (robot description, xacro)
@@ -19,11 +19,14 @@
   <!-- IMU -->
   <xacro:add_to_base_link_no_mesh element="imu">
-    <origin rpy="0 0 3.14" xyz="-0.35 0.1 -0.2"/>
+    <!-- The original transformation was: -->
+ 	  <origin rpy="0 0 -1.57" xyz="-0.35 0.1 -0.2"/>
+     <!-- good (real): use this one for calibration branch: -->
+		<!-- <origin rpy="0 0 3.14" xyz="-0.35 0.1 -0.2"/> -->
   </xacro:add_to_base_link_no_mesh>
-    <!-- IMU aligned with robot axis.
-       This frame is where the data of the IMU filter is published -->
-  <xacro:add_to_base_link_no_mesh element="imu_filter">
+  <!-- IMU aligned with robot axis.
+  This frame is where the data of the IMU filter is published -->
+  <!-- <xacro:add_to_base_link_no_mesh element="imu_filter">
     <origin rpy="0 0 0" xyz="-0.35 0.1 -0.2"/>
-  </xacro:add_to_base_link_no_mesh>
+  </xacro:add_to_base_link_no_mesh> -->
   <!-- USBL -->
   <!-- <xacro:add_to_base_link_no_mesh element="usbl">

Commit message: update xiroi_description files

File: urdf/core.urdf.xacro (robot description, xacro)
@@ -3,5 +3,5 @@
 <robot xmlns:xacro="http://www.ros.org/wiki/xacro">
   <!-- Load macros -->
-  <xacro:include filename="$(find cola2_lib)/src/cola2_lib/rosutils/urdf_macros.xacro"/>
+  <xacro:include filename="$(find cola2_lib_ros)/src/cola2_lib_ros/urdf_macros.xacro"/>
   <!-- Base link -->
   <link name="$(arg robot_namespace)/base_link">
@@ -13,30 +13,23 @@
     </visual>
   </link>
-  <!-- GPS -->
+  <!-- usbl -->
+  <xacro:add_to_base_link_no_mesh element="usbl">
+    <origin rpy="0 0 0" xyz="0.32 0 0.8"/>
+  </xacro:add_to_base_link_no_mesh>
+  <!-- gps -->
   <xacro:add_to_base_link_no_mesh element="gps">
     <origin rpy="0 0 0" xyz="0.70 0.35 -0.1"/>
   </xacro:add_to_base_link_no_mesh>
-  <!-- IMU -->
+  <!-- imu -->
   <xacro:add_to_base_link_no_mesh element="imu">
-    <!-- The original transformation was (use this for dev branch): -->
- 	  <origin rpy="0 0 -1.57" xyz="-0.35 0.1 -0.2"/>
-     <!-- good (real): use this one for calibration branch: -->
-		<!-- <origin rpy="0 0 3.14" xyz="-0.35 0.1 -0.2"/> -->
+    <origin rpy="0 0 -1.57" xyz="-0.35 0.1 -0.2"/>
   </xacro:add_to_base_link_no_mesh>
-  <!-- IMU aligned with robot axis.
-  This frame is where the data of the IMU filter is published -->
-  <!-- <xacro:add_to_base_link_no_mesh element="imu_filter">
-    <origin rpy="0 0 0" xyz="-0.35 0.1 -0.2"/>
-  </xacro:add_to_base_link_no_mesh> -->
-  <!-- USBL -->
-  <!-- <xacro:add_to_base_link_no_mesh element="usbl">
-    <origin rpy="0 0 0" xyz="0.32 0 0.8"/>
-  </xacro:add_to_base_link_no_mesh> -->
-  <!-- Thrusters -->
-  <xacro:add_thruster_no_mesh thruster_id="1">
+  <!-- thruster_0 -->
+  <xacro:add_to_base_link_no_mesh element="thruster_0">
     <origin xyz="-0.50 0.50 0.30" rpy="0 0 0" />
-  </xacro:add_thruster_no_mesh>
-  <xacro:add_thruster_no_mesh thruster_id="2">
+  </xacro:add_to_base_link_no_mesh>
+  <!-- thruster_1 -->
+  <xacro:add_to_base_link_no_mesh element="thruster_1">
     <origin xyz="-0.50 -0.50 0.30" rpy="0 0 0" />
-  </xacro:add_thruster_no_mesh>
+  </xacro:add_to_base_link_no_mesh>
 </robot>

File: urdf/payload.urdf.xacro (robot description, xacro)
@@ -5,17 +5,8 @@
     The robot_namespace argument has to be set mandatory by the user when calling the xacro
     file or using the following line to set it as default.
-    xacro:arg name="robot_namespace" default="sparus2"/
+    <xacro:arg name="robot_namespace" default="sparus2"/>
   -->
-  <!-- <xacro:arg name="robot_xacro" default="$(find sparus2_description)/urdf/core.urdf.xacro"/> -->
   <xacro:arg name="robot_xacro" default="$(find xiroi_description)/urdf/core.urdf.xacro"/>
-  <!-- Load basic Xiroi urdf -->
+  <!-- Load basic XiroiII urdf -->
   <xacro:include filename="$(arg robot_xacro)"/>
-  <!-- USBL -->
-  <xacro:add_to_base_link_no_mesh element="usbl">
-    <origin rpy="0 0 0" xyz="0.32 0 0.8"/>
-  </xacro:add_to_base_link_no_mesh>
-  <!-- Cameras
-  <xacro:add_to_base_link_no_mesh element="multibeam">
-    <origin rpy="0 -${pi/2} ${pi}" xyz="0.5 0 0"/>
-  </xacro:add_to_base_link_no_mesh>-->
 </robot>
